Commit message: Include lds01 mesh and first-guess position

File: urdf/homey.urdf.xacro (robot description, xacro)
@@ -1,4 +1,4 @@
 <?xml version="1.0"?>
-<robot name="turtlebot" xmlns:xacro="http://ros.org/wiki/xacro">
+<robot name="homey" xmlns:xacro="http://ros.org/wiki/xacro">
   <xacro:include filename="$(find turtlebot_description)/urdf/turtlebot_common_library.urdf.xacro" />
   <xacro:include filename="$(find kobuki_description)/urdf/kobuki.urdf.xacro" />
@@ -6,3 +6,28 @@
   <xacro:kobuki/>
   <xacro:stack_hexagons parent="base_link"/>
+  <joint name="scan_joint" type="fixed">
+    <parent link="base_link"/>
+    <child link="base_scan"/>
+    <origin xyz="0.05 0 0.221" rpy="0 0 3.14"/>
+  </joint>
+  <link name="base_scan">
+    <visual>
+      <origin xyz="0 0 0.0" rpy="0 0 0"/>
+      <geometry>
+        <mesh filename="package://robot_stack/meshes/lds01.stl" scale="0.001 0.001 0.001"/>
+      </geometry>
+      <material name="dark"/>
+    </visual>
+    <collision>
+      <origin xyz="0.015 0 -0.0065" rpy="0 0 0"/>
+      <geometry>
+        <cylinder length="0.0315" radius="0.055"/>
+      </geometry>
+    </collision>
+    <inertial>
+      <mass value="0.114" />
+      <origin xyz="0 0 0" />
+      <inertia ixx="0.001" ixy="0.0" ixz="0.0" iyy="0.001" iyz="0.0" izz="0.001" />
+    </inertial>
+  </link>
 </robot>

Commit message: Add gazebo laser sim to kobuki model

File: urdf/homey.urdf.xacro (robot description, xacro)
@@ -6,10 +6,10 @@
   <xacro:kobuki/>
   <xacro:stack_hexagons parent="base_link"/>
-  <joint name="scan_joint" type="fixed">
+  <joint name="laser_joint" type="fixed">
     <parent link="base_link"/>
-    <child link="base_scan"/>
+    <child link="laser_link"/>
     <origin xyz="0.05 0 0.221" rpy="0 0 3.14"/>
   </joint>
-  <link name="base_scan">
+  <link name="laser_link">
     <visual>
       <origin xyz="0 0 0.0" rpy="0 0 0"/>
@@ -31,3 +31,37 @@
     </inertial>
   </link>
+  <gazebo reference="laser_link">
+    <sensor type="ray" name="laser">
+      <plugin name="gazebo_ros_laser_controller" filename="libgazebo_ros_ray_sensor.so">
+        <ros>
+          <argument>~/out:=scan</argument>
+        </ros>
+        <output_type>sensor_msgs/LaserScan</output_type>
+        <frame_name>laser_link</frame_name>
+      </plugin>
+      <always_on>true</always_on>
+      <update_rate>5</update_rate>
+      <visualize>true</visualize>
+      <ray>
+        <scan>
+          <horizontal>
+            <samples>360</samples>
+            <resolution>1</resolution>
+            <min_angle>${-M_PI}</min_angle>
+            <max_angle>${M_PI}</max_angle>
+          </horizontal>
+        </scan>
+        <range>
+          <min>0.2</min>
+          <max>5</max>
+          <resolution>1</resolution>
+        </range>
+        <noise>
+          <type>gaussian</type>
+          <mean>0.0</mean>
+          <stddev>0.0</stddev>
+        </noise>
+      </ray>
+    </sensor>
+  </gazebo>
 </robot>
